Commit message: Lidar added

File: description/robot.urdf.xacro (robot description, xacro)
@@ -2,3 +2,5 @@
 <robot xmlns:xacro="http://www.ros.org/wiki/xacro"  name="robot">
     <xacro:include filename="$(find prac_bot)/description/robot_core.xacro" />
+    <xacro:include filename="$(find prac_bot)/description/gazebo_control.xacro" />
+    <xacro:include filename="$(find prac_bot)/description/lidar.xacro" />
 </robot>

File: description/robot_core.xacro (robot description, xacro)
@@ -14,4 +14,7 @@
     <material name="orange">
         <color rgba="1.0 0.5 0.0 1.0" />
+    </material>
+    <material name="red">
+        <color rgba="1.0 0.0 0.0 1.0" />
     </material>
     <!-- Base Link -->
@@ -42,4 +45,7 @@
         </xacro:inertial_box>
     </link>
+    <gazebo reference="chassis">
+        <material>Gazebo/White</material>
+    </gazebo>
     <!-- Left Wheel Link -->
     <joint name="left_wheel_joint" type="continuous">
@@ -65,4 +71,7 @@
         </xacro:inertial_cylinder>
     </link>
+    <gazebo reference="left_wheel">
+        <material>Gazebo/Blue</material>
+    </gazebo>
     <!-- Right Wheel Link -->
     <joint name="right_wheel_joint" type="continuous">
@@ -88,4 +97,7 @@
         </xacro:inertial_cylinder>
     </link>
+    <gazebo reference="right_wheel">
+        <material>Gazebo/Blue</material>
+    </gazebo>
     <!-- Caster Wheel Link -->
     <joint name="caster_wheel_joint" type="fixed">
@@ -110,3 +122,8 @@
         </xacro:inertial_sphere>
     </link>
+    <gazebo reference="caster_wheel">
+        <material>Gazebo/Black</material>
+        <mu1>0.01</mu1>
+        <mu2>0.01</mu2>
+    </gazebo>
 </robot>
