Commit message: Remove old RViz configuration and update simulation launch files; add lidar and joint state publisher configurations.

File: description/gazebo_control.xacro (robot description, xacro)
@@ -7,8 +7,8 @@
         <right_joint>right_wheel_joint</right_joint>
         <!-- Kinematics -->
-        <wheel_separation>0.35</wheel_separation>
-        <wheel_radius>0.05</wheel_radius>
+        <wheel_separation>0.297</wheel_separation>
+        <wheel_radius>0.033</wheel_radius>
         <!-- Limits -->
-        <max_linear_acceleration>10.0</max_linear_acceleration>
+        <max_linear_acceleration>0.33</max_linear_acceleration>
         <!-- Topics (override defaults) -->
         <topic>cmd_vel</topic>
@@ -19,10 +19,15 @@
         <child_frame_id>base_link</child_frame_id>
         <robot_base_frame>base_link</robot_base_frame>
+        <odom_publisher_frequency>30.0</odom_publisher_frequency>
         <publish_odom>true</publish_odom>
         <publish_odom_tf>true</publish_odom_tf>
         <publish_wheel_tf>true</publish_wheel_tf>
     </plugin>
+    <plugin filename="gz-sim-joint-state-publisher-system" name="gz::sim::systems::JointStatePublisher">
+        <topic>joint_states</topic>
+        <joint_names>left_wheel_joint right_wheel_joint</joint_names>
+    </plugin>
     <plugin filename="gz-sim-sensors-system" name="gz::sim::systems::Sensors">
-        <render_engine>ogre</render_engine>
+        <render_engine>ogre2</render_engine>
     </plugin>
 </gazebo>

File: description/lidar.xacro (robot description, xacro)
@@ -4,5 +4,5 @@
         <parent link="chassis" />
         <child link="lidar" />
-        <origin xyz="0.15 0 0.175" rpy="0 0 0" />
+        <origin xyz="0.122 0 0.212" rpy="0 0 0" />
     </joint>
     <link name="lidar">
@@ -10,4 +10,11 @@
             <geometry>
                 <cylinder radius="0.05" length="0.04" />
+            </geometry>
+            <material name="red"/>
+        </visual>
+        <visual>
+            <origin xyz="0 0 -0.05" />
+            <geometry>
+                <cylinder radius="0.01" length="0.1" />
             </geometry>
             <material name="red"/>
@@ -32,5 +39,4 @@
                     <horizontal>
                         <samples>360</samples>
-                        <resolution>1</resolution>
                         <min_angle>-3.14159</min_angle>
                         <max_angle>3.14159</max_angle>
@@ -42,4 +48,5 @@
                 </range>
             </lidar>
+            <gz_frame_id>lidar</gz_frame_id>
             <always_on>true</always_on>
             <visualize>true</visualize>
